File: keyboard/keyboard.sch (KiCad schematic (older format))
At the start: 2 parts

Commit message: update
Parts:
- removed J?: Conn_01x08_Female, symbol Connector:Conn_01x08_Female
- added J2: Conn_01x08_Male, Connector_PinHeader_2.54mm:PinHeader_1x08_P2.54mm_Vertical, symbol Connector:Conn_01x08_Male
- added J3: Conn_01x05_Male, Connector_PinSocket_2.54mm:PinSocket_1x05_P2.54mm_Vertical, symbol Connector:Conn_01x05_Male
- added J4, J5: Conn_01x14_Male, Connector_PinSocket_2.54mm:PinSocket_1x14_P2.54mm_Vertical, symbol Connector:Conn_01x14_Male
- added J6: Conn_02x07_Top_Bottom, Connector_PinSocket_2.54mm:PinSocket_2x07_P2.54mm_Vertical, symbol Connector_Generic:Conn_02x07_Top_Bottom
- added U1: Teensy3.2, teensy:Teensy30_31_32_LC, symbol teensy:Teensy3.2
- J1: renamed from J?; footprint (none) -> custom:Con_FFC_28_ALT
Connections:
- net labels added: A_12, GND_PAD
- wire segments 0 -> 107

Commit message: added traces
Parts:
- added J7: Conn_01x28_Male, custom:Heade2.54m_28pin, symbol Connector:Conn_01x28_Male
- added J8: Conn_01x08_Female, Connector_PinHeader_2.54mm:PinHeader_1x08_P2.54mm_Vertical, symbol Connector:Conn_01x08_Female
- J6: footprint Connector_PinSocket_2.54mm:PinSocket_2x07_P2.54mm_Vertical -> custom:PinHeader_2x07Custom
Connections:
- wire segments 107 -> 135
Changed lines of the file:
@@
 F 0 "J6" H 10150 2467 50  0000 C CNN
 F 1 "Conn_02x07_Top_Bottom" H 10150 2376 50  0000 C CNN
-F 2 "Connector_PinSocket_2.54mm:PinSocket_2x07_P2.54mm_Vertical" H 10100 1950 50  0001 C CNN
+F 2 "custom:PinHeader_2x07Custom" H 10100 1950 50  0001 C CNN
 F 3 "~" H 10100 1950 50  0001 C CNN
 	1    10100 1950
 	1    0    0    -1
 $EndComp
+$Comp
+L Connector:Conn_01x28_Male J7
+U 1 1 5D57E484
+P 3300 2600
+F 0 "J7" H 3273 2480 50  0000 R CNN
+F 1 "Conn_01x28_Male" H 3273 2571 50  0000 R CNN
+F 2 "custom:Heade2.54m_28pin" H 3300 2600 50  0001 C CNN
+F 3 "~" H 3300 2600 50  0001 C CNN
+	1    3300 2600
+	-1   0    0    1
+$EndComp
+$Comp
+L Connector:Conn_01x08_Female J8
+U 1 1 5D57E64C
+P 2850 4700
+F 0 "J8" H 2877 4676 50  0000 L CNN
+F 1 "Conn_01x08_Female" H 2877 4585 50  0000 L CNN
+F 2 "Connector_PinHeader_2.54mm:PinHeader_1x08_P2.54mm_Vertical" H 2850 4700 50  0001 C CNN
+F 3 "~" H 2850 4700 50  0001 C CNN
+	1    2850 4700
+	1    0    0    -1
+$EndComp
+Wire Wire Line
+	3100 1200 2600 1200
+Wire Wire Line
+	3100 1300 2600 1300
+Wire Wire Line
+	3100 1400 2600 1400
+Wire Wire Line
+	2600 1500 3100 1500
+Wire Wire Line
+	3100 1600 2600 1600
+Wire Wire Line
+	2600 1700 3100 1700
+Wire Wire Line
+	3100 1800 2600 1800
+Wire Wire Line
+	3100 1900 2600 1900
+Wire Wire Line
+	2600 2000 3100 2000
+Wire Wire Line
+	3100 2100 2600 2100
+Wire Wire Line
+	2600 2200 3100 2200
+Wire Wire Line
+	2600 2300 3100 2300
+Wire Wire Line
+	3100 2400 2600 2400
+Wire Wire Line
+	2600 2500 3100 2500
+Wire Wire Line
+	3100 2600 2600 2600
+Wire Wire Line
+	2600 2700 3100 2700
+Wire Wire Line
+	3100 2800 2600 2800
+Wire Wire Line
+	2600 2900 3100 2900
+Wire Wire Line
+	3100 3000 2600 3000
+Wire Wire Line
+	2600 3100 3100 3100
+Wire Wire Line
+	3100 3200 2600 3200
+Wire Wire Line
+	2600 3300 3100 3300
+Wire Wire Line
+	3100 3400 2600 3400
+Wire Wire Line
+	3100 3500 2600 3500
+Wire Wire Line
+	2600 3600 3100 3600
+Wire Wire Line
+	3100 3700 2600 3700
+Wire Wire Line
+	2600 3800 3100 3800
+Wire Wire Line
+	2600 3900 3100 3900
 $EndSCHEMATC

Commit message: pcb layout
Parts:
- added J10: Conn_01x03_Male, Connector_PinSocket_2.54mm:PinSocket_1x03_P2.54mm_Vertical, symbol Connector:Conn_01x03_Male
- added J9: Conn_01x01_Male, Connector_PinHeader_2.54mm:PinHeader_1x01_P2.54mm_Vertical, symbol Connector:Conn_01x01_Male
Connections:
- wire segments 135 -> 139
Changed lines of the file:
@@
 Wire Wire Line
 	2600 3900 3100 3900
+$Comp
+L Connector:Conn_01x01_Male J9
+U 1 1 5D5AAF5C
+P 9950 3650
+F 0 "J9" H 9923 3580 50  0000 R CNN
+F 1 "Conn_01x01_Male" H 9923 3671 50  0000 R CNN
+F 2 "Connector_PinHeader_2.54mm:PinHeader_1x01_P2.54mm_Vertical" H 9950 3650 50  0001 C CNN
+F 3 "~" H 9950 3650 50  0001 C CNN
+	1    9950 3650
+	-1   0    0    1
+$EndComp
+Wire Wire Line
+	8950 3650 9750 3650
+$Comp
+L Connector:Conn_01x03_Male J10
+U 1 1 5D5BD521
+P 9450 3450
+F 0 "J10" H 9423 3380 50  0000 R CNN
+F 1 "Conn_01x03_Male" H 9423 3471 50  0000 R CNN
+F 2 "Connector_PinSocket_2.54mm:PinSocket_1x03_P2.54mm_Vertical" H 9450 3450 50  0001 C CNN
+F 3 "~" H 9450 3450 50  0001 C CNN
+	1    9450 3450
+	-1   0    0    1
+$EndComp
+Wire Wire Line
+	9250 3350 8950 3350
+Wire Wire Line
+	8950 3450 9250 3450
+Wire Wire Line
+	9250 3550 8950 3550
 $EndSCHEMATC

Commit message: changed mcu to teensy++
Parts:
- removed J10: Conn_01x03_Male, Connector_PinSocket_2.54mm:PinSocket_1x03_P2.54mm_Vertical, symbol Connector:Conn_01x03_Male
- removed J3: Conn_01x05_Male, Connector_PinSocket_2.54mm:PinSocket_1x05_P2.54mm_Vertical, symbol Connector:Conn_01x05_Male
- removed J4, J5: Conn_01x14_Male, Connector_PinSocket_2.54mm:PinSocket_1x14_P2.54mm_Vertical, symbol Connector:Conn_01x14_Male
- removed J6: Conn_02x07_Top_Bottom, custom:PinHeader_2x07Custom, symbol Connector_Generic:Conn_02x07_Top_Bottom
- removed J9: Conn_01x01_Male, Connector_PinHeader_2.54mm:PinHeader_1x01_P2.54mm_Vertical, symbol Connector:Conn_01x01_Male
- removed U1: Teensy3.2, teensy:Teensy30_31_32_LC, symbol teensy:Teensy3.2
- added J? (x2): Conn_01x20_Male, symbol Connector:Conn_01x20_Male
- added U?: Teensy++2.0, symbol teensy:Teensy++2.0
Connections:
- net labels removed: A_12, GND_PAD
- wire segments 139 -> 79

Commit message: switched to teensy ++ 2.0
Parts:
- added J10: Conn_01x01_Male, Connector_PinHeader_2.54mm:PinHeader_1x01_P2.54mm_Vertical, symbol Connector:Conn_01x01_Male
- added J5: Conn_01x03_Female, Connector_PinHeader_2.54mm:PinHeader_1x03_P2.54mm_Vertical, symbol Connector:Conn_01x03_Female
- added J6, J9: Conn_01x04_Male, Connector_PinHeader_2.54mm:PinHeader_1x04_P2.54mm_Vertical, symbol Connector:Conn_01x04_Male
- J3, J4: renamed from J?; footprint (none) -> Connector_PinHeader_2.54mm:PinHeader_1x20_P2.54mm_Vertical
- U1: renamed from U?; footprint (none) -> teensy:Teensy2.0++
Connections:
- wire segments 79 -> 98
Changed lines of the file:
@@
 	2600 3900 3100 3900
 $Comp
-L teensy:Teensy++2.0 U?
+L teensy:Teensy++2.0 U1
 U 1 1 5D60E247
 P 7650 2800
-F 0 "U?" H 7650 4237 60  0000 C CNN
+F 0 "U1" H 7650 4237 60  0000 C CNN
 F 1 "Teensy++2.0" H 7650 4131 60  0000 C CNN
-F 2 "" H 7750 1950 60  0000 C CNN
+F 2 "teensy:Teensy2.0++" H 7750 1950 60  0001 C CNN
 F 3 "" H 7750 1950 60  0000 C CNN
 	1    7650 2800
@@
 $EndComp
 $Comp
-L Connector:Conn_01x20_Male J?
+L Connector:Conn_01x20_Male J3
 U 1 1 5D6211A9
 P 5550 2550
-F 0 "J?" H 5656 3628 50  0000 C CNN
+F 0 "J3" H 5656 3628 50  0000 C CNN
 F 1 "Conn_01x20_Male" H 5656 3537 50  0000 C CNN
-F 2 "" H 5550 2550 50  0001 C CNN
+F 2 "Connector_PinHeader_2.54mm:PinHeader_1x20_P2.54mm_Vertical" H 5550 2550 50  0001 C CNN
 F 3 "~" H 5550 2550 50  0001 C CNN
 	1    5550 2550
@@
 	8550 4450 9050 4450
 $Comp
-L Connector:Conn_01x20_Male J?
+L Connector:Conn_01x20_Male J4
 U 1 1 5D695126
 P 9250 3550
-F 0 "J?" H 9223 3430 50  0000 R CNN
+F 0 "J4" H 9223 3430 50  0000 R CNN
 F 1 "Conn_01x20_Male" H 9223 3521 50  0000 R CNN
-F 2 "" H 9250 3550 50  0001 C CNN
+F 2 "Connector_PinHeader_2.54mm:PinHeader_1x20_P2.54mm_Vertical" H 9250 3550 50  0001 C CNN
 F 3 "~" H 9250 3550 50  0001 C CNN
 	1    9250 3550
@@
 Wire Wire Line
 	6950 3550 5750 3550
+$Comp
+L Connector:Conn_01x03_Female J5
+U 1 1 5D68E209
+P 5950 4200
+F 0 "J5" H 5844 3875 50  0000 C CNN
+F 1 "Conn_01x03_Female" H 5844 3966 50  0000 C CNN
+F 2 "Connector_PinHeader_2.54mm:PinHeader_1x03_P2.54mm_Vertical" H 5950 4200 50  0001 C CNN
+F 3 "~" H 5950 4200 50  0001 C CNN
+	1    5950 4200
+	-1   0    0    1
+$EndComp
+Wire Wire Line
+	6950 3650 6500 3650
+Wire Wire Line
+	6500 3650 6500 4100
+Wire Wire Line
+	6500 4100 6150 4100
+Wire Wire Line
+	6950 3750 6600 3750
+Wire Wire Line
+	6600 3750 6600 4200
+Wire Wire Line
+	6600 4200 6150 4200
+Wire Wire Line
+	6950 3850 6700 3850
+Wire Wire Line
+	6700 3850 6700 4300
+Wire Wire Line
+	6700 4300 6150 4300
+$Comp
+L Connector:Conn_01x04_Male J6
+U 1 1 5D6A8E75
+P 9250 1950
+F 0 "J6" H 9223 1830 50  0000 R CNN
+F 1 "Conn_01x04_Male" H 9223 1921 50  0000 R CNN
+F 2 "Connector_PinHeader_2.54mm:PinHeader_1x04_P2.54mm_Vertical" H 9250 1950 50  0001 C CNN
+F 3 "~" H 9250 1950 50  0001 C CNN
+	1    9250 1950
+	-1   0    0    1
+$EndComp
+Wire Wire Line
+	8350 1750 9050 1750
+Wire Wire Line
+	9050 1850 8350 1850
+Wire Wire Line
+	8350 1950 9050 1950
+Wire Wire Line
+	8350 2050 9050 2050
+$Comp
+L Connector:Conn_01x04_Male J9
+U 1 1 5D6B41AA
+P 9250 2350
+F 0 "J9" H 9223 2230 50  0000 R CNN
+F 1 "Conn_01x04_Male" H 9223 2321 50  0000 R CNN
+F 2 "Connector_PinHeader_2.54mm:PinHeader_1x04_P2.54mm_Vertical" H 9250 2350 50  0001 C CNN
+F 3 "~" H 9250 2350 50  0001 C CNN
+	1    9250 2350
+	-1   0    0    1
+$EndComp
+Wire Wire Line
+	8350 2150 9050 2150
+Wire Wire Line
+	8350 2250 9050 2250
+Wire Wire Line
+	9050 2350 8350 2350
+Wire Wire Line
+	8350 2450 9050 2450
+$Comp
+L Connector:Conn_01x01_Male J10
+U 1 1 5D6C08B6
+P 9400 1600
+F 0 "J10" H 9373 1530 50  0000 R CNN
+F 1 "Conn_01x01_Male" H 9373 1621 50  0000 R CNN
+F 2 "Connector_PinHeader_2.54mm:PinHeader_1x01_P2.54mm_Vertical" H 9400 1600 50  0001 C CNN
+F 3 "~" H 9400 1600 50  0001 C CNN
+	1    9400 1600
+	-1   0    0    1
+$EndComp
+Wire Wire Line
+	9200 1600 8350 1600
+Wire Wire Line
+	8350 1600 8350 1650
 $EndSCHEMATC

Commit message: replaced with correct 30 pin ffc
Parts:
- removed J1: Conn_01x28_Female, custom:Con_FFC_28_ALT, symbol Connector:Conn_01x28_Female
- removed J7: Conn_01x28_Male, custom:Heade2.54m_28pin, symbol Connector:Conn_01x28_Male
- added J1: Conn_01x30_Female, custom:Con_FFC_30_2.0mm, symbol Connector:Conn_01x30_Female
- added J7: Conn_01x30_Male, custom:Heade2.54m_30pin_working, symbol Connector:Conn_01x30_Male
Connections:
- wire segments 98 -> 100
Changed lines of the file:
@@
 $EndDescr
-$Comp
-L Connector:Conn_01x28_Female J1
-U 1 1 5D3FD40F
-P 2400 2600
-F 0 "J1" H 2427 2576 50  0000 L CNN
-F 1 "Conn_01x28_Female" H 2427 2485 50  0000 L CNN
-F 2 "custom:Con_FFC_28_ALT" H 2400 2600 50  0001 C CNN
-F 3 "~" H 2400 2600 50  0001 C CNN
-	1    2400 2600
-	-1   0    0    1
-$EndComp
 $Comp
 L Connector:Conn_01x08_Male J2
@@
 $EndComp
 $Comp
-L Connector:Conn_01x28_Male J7
-U 1 1 5D57E484
-P 3300 2600
-F 0 "J7" H 3273 2480 50  0000 R CNN
-F 1 "Conn_01x28_Male" H 3273 2571 50  0000 R CNN
-F 2 "custom:Heade2.54m_28pin" H 3300 2600 50  0001 C CNN
-F 3 "~" H 3300 2600 50  0001 C CNN
-	1    3300 2600
-	-1   0    0    1
-$EndComp
-$Comp
 L Connector:Conn_01x08_Female J8
 U 1 1 5D57E64C
@@
 	3100 2800 2600 2800
 Wire Wire Line
-	2600 2900 3100 2900
-Wire Wire Line
 	3100 3000 2600 3000
 Wire Wire Line
@@
 Wire Wire Line
 	2600 3800 3100 3800
-Wire Wire Line
-	2600 3900 3100 3900
 $Comp
 L teensy:Teensy++2.0 U1
@@
 Wire Wire Line
 	8350 1600 8350 1650
+Wire Wire Line
+	2600 2900 3100 2900
+Wire Wire Line
+	3100 1100 2600 1100
+Wire Wire Line
+	2600 1000 3100 1000
+Wire Wire Line
+	3100 900  2600 900
+$Comp
+L Connector:Conn_01x30_Female J1
+U 1 1 5E73DEF3
+P 2400 2400
+F 0 "J1" H 2294 675 50  0000 C CNN
+F 1 "Conn_01x30_Female" H 2294 766 50  0000 C CNN
+F 2 "custom:Con_FFC_30_2.0mm" H 2400 2400 50  0001 C CNN
+F 3 "~" H 2400 2400 50  0001 C CNN
+	1    2400 2400
+	-1   0    0    1
+$EndComp
+$Comp
+L Connector:Conn_01x30_Male J7
+U 1 1 5E73DFB5
+P 3300 2400
+F 0 "J7" H 3273 2280 50  0000 R CNN
+F 1 "Conn_01x30_Male" H 3273 2371 50  0000 R CNN
+F 2 "custom:Heade2.54m_30pin_working" H 3300 2400 50  0001 C CNN
+F 3 "~" H 3300 2400 50  0001 C CNN
+	1    3300 2400
+	-1   0    0    1
+$EndComp
 $EndSCHEMATC
