File: keyboard/keyboard.kicad_pcb (KiCad board)
At the start: 2 copper layers, 7 parts, among them J1 Conn_01x28_Female, J2 Conn_01x08_Male, J3 Conn_01x05_Male, J4 Conn_01x14_Male, J5 Conn_01x14_Male, J6 Conn_02x07_Top_Bottom, U1 Teensy3.2

Commit message: added traces
Parts:
- added J7: Conn_01x28_Male, custom:Heade2.54m_28pin, F.Cu at (218.6, 69.5)
- added J8: Conn_01x08_Female, Connector_PinHeader_2.54mm:PinHeader_1x08_P2.54mm_Vertical, F.Cu at (180.3, 78.0)
- J6: footprint Connector_PinSocket_2.54mm:PinSocket_2x07_P2.54mm_Vertical -> custom:PinHeader_2x07Custom; moved to B.Cu
- moved J1 98.0 mm to (233.9, 95.0), turned to 180 degrees
- moved J6 55.3 mm to (219.8, 136.8), turned to 90 degrees
- moved J5 25.1 mm to (187.3, 120.8)
- moved J2 23.4 mm to (168.4, 77.9)
- moved J4 20.3 mm to (154.3, 151.0)
- moved U1 18.4 mm to (170.8, 136.5)
- moved J3 17.3 mm to (212.0, 154.9)
Routing:
- net Net-(J1-Pad15): track 0.00 -> 66.4 mm
- net Net-(J1-Pad13): track 0.00 -> 62.6 mm
- net /A_12: track 0.00 -> 61.9 mm
- net Net-(J1-Pad17): track 0.00 -> 60.0 mm
- net Net-(J6-Pad3): track 0.00 -> 58.4 mm
- net Net-(J1-Pad11): track 0.00 -> 56.2 mm
- net /GND_PAD: track 0.00 -> 55.6 mm
- net Net-(J1-Pad19): track 0.00 -> 53.4 mm
- net Net-(J6-Pad4): track 0.00 -> 53.0 mm
- net Net-(J1-Pad9): track 0.00 -> 49.8 mm
- net Net-(J6-Pad8): track 0.00 -> 49.6 mm
- net Net-(J6-Pad5): track 0.00 -> 47.9 mm
- net Net-(J1-Pad21): track 0.00 -> 46.8 mm
- net Net-(J6-Pad9): track 0.00 -> 44.2 mm
- net Net-(J6-Pad6): track 0.00 -> 42.1 mm
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
Commit message: pcb layout
Parts:
- added J10: Conn_01x03_Male, Connector_PinSocket_2.54mm:PinSocket_1x03_P2.54mm_Vertical, F.Cu at (191.1, 102.0)
- added J9: Conn_01x01_Male, Connector_PinHeader_2.54mm:PinHeader_1x01_P2.54mm_Vertical, F.Cu at (185.5, 102.0)
- moved J4 99.7 mm to (190.1, 57.9), turned to 0 degrees
- moved J2 95.2 mm to (252.3, 122.8), turned to 270 degrees
- moved J8 91.6 mm to (252.2, 134.7), turned to 270 degrees
- moved U1 70.7 mm to (204.6, 74.4), turned to 270 degrees
- moved J3 47.1 mm to (186.2, 115.6), turned to 90 degrees
- moved J5 44.5 mm to (220.3, 90.9), turned to 180 degrees
- moved J6 20.4 mm to (204.3, 123.4), turned to 0 degrees
- moved J1 18.3 mm to (250.2, 86.6)
- moved J7 18.3 mm to (234.8, 61.1)
Routing:
- net Net-(J9-Pad1): track 0.00 -> 80.8 mm
- net Net-(J10-Pad1): track 0.00 -> 48.6 mm
- net Net-(J10-Pad2): track 0.00 -> 44.7 mm
- net Net-(J10-Pad3): track 0.00 -> 42.8 mm
Other:
- board outline added: 82.7 x 95.8 mm
- board text added: "1"
- board text added: "2"
- board text added: "27"
- board text added: "28"
- board text added: "28 Pin FFC Connector"
- board text added: "3.3v"
- board text added: "8"
- board text added: "A10"
- board text added: "A11"
- board text added: "A12"
- board text added: "A13"
- board text added: "A14"
- board text added: "AREF"
- board text added: "BY: Jonathan Low"
- board text added: "D12"
- board text added: "D13"
- board text added: "D24"
- board text added: "D25"
- board text added: "D26"
- board text added: "D27"
- board text added: "D28"
- board text added: "D29"
- board text added: "D30"
- board text added: "D31"
- board text added: "D32"
- board text added: "D33"
- board text added: "GND"
- board text added: "TP-Keyboard Test Board v1.0"
- board text added: "Teensy 3.2"
- board text added: "Track Point Module"
- board text added: "VBAT"
- board text added: "VIN"
- board text added: "VUSB"

Commit message: changed mcu to teensy++
Changed lines of the file:
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@@
     )
   )
-  (gr_text "BY: Jonathan Low" (at 189.611 143.256) (layer F.SilkS)
+  (gr_text "BY: Jonathan Low" (at 189.738 143.129) (layer F.SilkS)
     (effects (font (size 1.5 1.5) (thickness 0.3)))
   )
-  (gr_text "TP-Keyboard Test Board v1.0" (at 196.342 140.335) (layer F.SilkS)
+  (gr_text "TP-Keyboard Test Board v1.0" (at 196.469 140.208) (layer F.SilkS)
     (effects (font (size 1.5 1.5) (thickness 0.3)))
   )
-  (gr_text "Teensy 3.2" (at 185.039 126.365) (layer F.SilkS)
+  (gr_text "Teensy 3.2" (at 204.851 96.774) (layer F.SilkS)
     (effects (font (size 1.5 1.5) (thickness 0.3)))
   )
-  (gr_text "Track Point Module" (at 241.808 145.542) (layer F.SilkS)
+  (gr_text "Track Point Module" (at 243.459 141.351) (layer F.SilkS)
     (effects (font (size 1.5 1.5) (thickness 0.3)))
   )

Commit message: switched to teensy ++ 2.0
Parts:
- J10: value Conn_01x03_Male -> Conn_01x01_Male; footprint Connector_PinSocket_2.54mm:PinSocket_1x03_P2.54mm_Vertical -> Connector_PinHeader_2.54mm:PinHeader_1x01_P2.54mm_Vertical
- J3: value Conn_01x05_Male -> Conn_01x20_Male; footprint Connector_PinSocket_2.54mm:PinSocket_1x05_P2.54mm_Vertical -> Connector_PinHeader_2.54mm:PinHeader_1x20_P2.54mm_Vertical
- J4: value Conn_01x14_Male -> Conn_01x20_Male; footprint Connector_PinSocket_2.54mm:PinSocket_1x14_P2.54mm_Vertical -> Connector_PinHeader_2.54mm:PinHeader_1x20_P2.54mm_Vertical
- J5: value Conn_01x14_Male -> Conn_01x03_Female; footprint Connector_PinSocket_2.54mm:PinSocket_1x14_P2.54mm_Vertical -> Connector_PinHeader_2.54mm:PinHeader_1x03_P2.54mm_Vertical
- J6: value Conn_02x07_Top_Bottom -> Conn_01x04_Male; footprint custom:PinHeader_2x07Custom -> Connector_PinHeader_2.54mm:PinHeader_1x04_P2.54mm_Vertical; moved to F.Cu
- J9: value Conn_01x01_Male -> Conn_01x04_Male; footprint Connector_PinHeader_2.54mm:PinHeader_1x01_P2.54mm_Vertical -> Connector_PinHeader_2.54mm:PinHeader_1x04_P2.54mm_Vertical
- U1: value Teensy3.2 -> Teensy++2.0; footprint teensy:Teensy30_31_32_LC -> teensy:Teensy2.0++
- moved J4 58.4 mm to (219.7, 108.2), turned to 180 degrees
- moved J3 55.6 mm to (184.9, 59.9), turned to 0 degrees
- moved J9 37.9 mm to (216.4, 124.0)
- moved J5 31.7 mm to (204.1, 118.1), turned to 270 degrees
- moved J10 15.9 mm to (184.9, 116.6), turned to 0 degrees
- moved J6 13.7 mm to (190.6, 123.6)
- moved U1 10.1 mm to (201.5, 84.1)
Connections:
- J6 pad 1: /A_12 -> Net-(J6-Pad1)
- J6 pad 2: /GND_PAD -> Net-(J6-Pad2)
- U1 pad 1: Net-(J4-Pad1) -> Net-(J3-Pad1)
- U1 pad 10: Net-(J4-Pad10) -> Net-(J3-Pad10)
- U1 pad 11: Net-(J4-Pad11) -> Net-(J3-Pad11)
- U1 pad 12: Net-(J4-Pad12) -> Net-(J3-Pad12)
- U1 pad 13: Net-(J4-Pad13) -> Net-(J3-Pad13)
- U1 pad 14: Net-(J4-Pad14) -> Net-(J3-Pad14)
- U1 pad 15: Net-(J3-Pad1) -> Net-(J3-Pad15)
- U1 pad 16: Net-(J3-Pad2) -> Net-(J3-Pad16)
- U1 pad 17: Net-(J3-Pad3) -> Net-(J3-Pad17)
- U1 pad 18: Net-(J3-Pad4) -> Net-(J3-Pad18)
- U1 pad 19: Net-(J3-Pad5) -> Net-(J3-Pad19)
- U1 pad 2: Net-(J4-Pad2) -> Net-(J3-Pad2)
- U1 pad 20: Net-(J5-Pad1) -> Net-(J3-Pad20)
- U1 pad 21: Net-(J5-Pad2) -> Net-(J5-Pad3)
- U1 pad 22: Net-(J5-Pad3) -> Net-(J5-Pad2)
- U1 pad 23: Net-(J5-Pad4) -> Net-(J5-Pad1)
- U1 pad 24: Net-(J5-Pad5) -> Net-(J4-Pad1)
- U1 pad 25: Net-(J5-Pad6) -> Net-(J4-Pad2)
- U1 pad 26: Net-(J5-Pad7) -> Net-(J4-Pad3)
- U1 pad 27: Net-(J5-Pad8) -> Net-(J4-Pad4)
- U1 pad 28: Net-(J5-Pad9) -> Net-(J4-Pad5)
- U1 pad 29: Net-(J5-Pad10) -> Net-(J4-Pad6)
- U1 pad 3: Net-(J4-Pad3) -> Net-(J3-Pad3)
- U1 pad 30: Net-(J5-Pad11) -> Net-(J4-Pad7)
- U1 pad 31: Net-(J5-Pad12) -> Net-(J4-Pad8)
- U1 pad 32: Net-(J5-Pad13) -> Net-(J4-Pad9)
- U1 pad 33: Net-(J5-Pad14) -> Net-(J4-Pad10)
- U1 pad 34: Net-(J9-Pad1) -> Net-(J4-Pad11)
- U1 pad 35: Net-(J10-Pad1) -> Net-(J4-Pad12)
- U1 pad 36: Net-(J10-Pad2) -> Net-(J4-Pad13)
- U1 pad 37: Net-(J10-Pad3) -> Net-(J4-Pad14)
- U1 pad 38: /A_12 -> Net-(J4-Pad15)
- U1 pad 39: /GND_PAD -> Net-(J4-Pad16)
- U1 pad 4: Net-(J4-Pad4) -> Net-(J3-Pad4)
- U1 pad 40: Net-(J6-Pad8) -> Net-(J4-Pad17)
- U1 pad 41: Net-(J6-Pad9) -> Net-(J4-Pad18)
- U1 pad 42: Net-(J6-Pad10) -> Net-(J4-Pad19)
- U1 pad 43: Net-(J6-Pad11) -> Net-(J4-Pad20)
- U1 pad 44: Net-(J6-Pad12) -> Net-(J9-Pad1)
- U1 pad 45: Net-(J6-Pad13) -> Net-(J9-Pad2)
- U1 pad 46: Net-(J6-Pad14) -> Net-(J9-Pad3)
- U1 pad 47: Net-(J6-Pad7) -> Net-(J9-Pad4)
- U1 pad 48: Net-(J6-Pad6) -> Net-(J6-Pad1)
- U1 pad 49: Net-(J6-Pad5) -> Net-(J6-Pad2)
- U1 pad 5: Net-(J4-Pad5) -> Net-(J3-Pad5)
- U1 pad 50: Net-(J6-Pad4) -> Net-(J6-Pad3)
- U1 pad 51: Net-(J6-Pad3) -> Net-(J6-Pad4)
- U1 pad 52: Net-(U1-Pad52) -> Net-(J10-Pad1)
- U1 pad 6: Net-(J4-Pad6) -> Net-(J3-Pad6)
- U1 pad 7: Net-(J4-Pad7) -> Net-(J3-Pad7)
- U1 pad 8: Net-(J4-Pad8) -> Net-(J3-Pad8)
- U1 pad 9: Net-(J4-Pad9) -> Net-(J3-Pad9)
Routing:
- net /A_12: track 61.9 -> 0.00 mm
- net /GND_PAD: track 55.6 -> 0.00 mm
- net Net-(J6-Pad8): track 49.6 -> 0.00 mm
- net Net-(J6-Pad5): track 47.9 -> 0.00 mm
- net Net-(J9-Pad1): track 80.8 -> 36.1 mm
- net Net-(J10-Pad2): track 44.7 -> 0.00 mm
- net Net-(J6-Pad9): track 44.2 -> 0.00 mm
- net Net-(J10-Pad3): track 42.8 -> 0.00 mm
- net Net-(J6-Pad6): track 42.1 -> 0.00 mm
- net Net-(J6-Pad1): track 0.00 -> 39.0 mm
- net Net-(J6-Pad2): track 0.00 -> 38.6 mm
- net Net-(J9-Pad4): track 0.00 -> 37.1 mm
- net Net-(J9-Pad3): track 0.00 -> 36.8 mm
- net Net-(J9-Pad2): track 0.00 -> 36.7 mm
- net Net-(J6-Pad7): track 36.7 -> 0.00 mm
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Other:
- board text added: "10"
- board text added: "11"
- board text added: "12"
- board text added: "13"
- board text added: "14"
- board text added: "15"
- board text added: "16"
- board text added: "17"
- board text added: "18"
- board text added: "19"
- board text added: "20"
- board text added: "21"
- board text added: "22"
- board text added: "23"
- board text added: "24"
- board text added: "25"
- board text added: "26"
- board text added: "3"
- board text added: "4"
- board text added: "5"
- board text added: "5V"
- board text added: "6"
- board text added: "7"
- board text added: "9"
- board text added: "ALE"
- board text added: "B0"
- board text added: "B1"
- board text added: "B2"
- board text added: "B3"
- board text added: "B4"
- board text added: "B5"
- board text added: "B6"
- board text added: "B7"
- board text added: "C0"
- board text added: "C1"
- board text added: "C2"
- board text added: "C3"
- board text added: "C4"
- board text added: "C5"
- board text added: "C6"
- board text added: "C7"
- board text added: "D0"
- board text added: "D1"
- board text added: "D2"
- board text added: "D3"
- board text added: "D4"
- board text added: "D5"
- board text added: "D6"
- board text added: "D7"
- board text added: "E0"
- board text added: "E1"
- board text added: "E6"
- board text added: "E7"
- board text added: "F0"
- board text added: "F1"
- board text added: "F2"
- board text added: "F3"
- board text added: "F4"
- board text added: "F5"
- board text added: "F6"
- board text added: "F7"
- board text added: "PA0"
- board text added: "PA1"
- board text added: "PA2"
- board text added: "PA3"
- board text added: "PA4"
- board text added: "PA5"
- board text added: "PA6"
- board text added: "PA7"
- board text added: "RST"
- board text added: "Teensy ++ 2.0"
- board text removed: "3.3v"
- board text removed: "A10"
- board text removed: "A11"
- board text removed: "A12"
- board text removed: "A13"
- board text removed: "A14"
- board text removed: "D12"
- board text removed: "D13"
- board text removed: "D24"
- board text removed: "D25"
- board text removed: "D26"
- board text removed: "D27"
- board text removed: "D28"
- board text removed: "D29"
- board text removed: "D30"
- board text removed: "D31"
- board text removed: "D32"
- board text removed: "D33"
- board text removed: "Teensy 3.2"
- board text removed: "VBAT"
- board text removed: "VIN"
- board text removed: "VUSB"

Commit message: fillets, mounting holes
Parts:
- added REF**: MountingHole_3.2mm_M3, MountingHole:MountingHole_3.2mm_M3, F.Cu at (257.4, 57.0)
- added REF**: MountingHole_3.2mm_M3, MountingHole:MountingHole_3.2mm_M3, F.Cu at (181.9, 57.0)
- added REF**: MountingHole_3.2mm_M3, MountingHole:MountingHole_3.2mm_M3, F.Cu at (181.9, 145.7)
- added REF**: MountingHole_3.2mm_M3, MountingHole:MountingHole_3.2mm_M3, F.Cu at (257.4, 145.7)
Other:
- outline, holes or cut-outs redrawn
Changed lines of the file:
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@@
   (general
     (thickness 1.6)
-    (drawings 137)
+    (drawings 139)
     (tracks 285)
     (zones 0)
-    (modules 11)
+    (modules 15)
     (nets 89)
   )
@@
     (descr "Through hole straight pin header, 1x14, 2.54mm pitch, single row")
     (tags "Through hole pin header THT 1x14 2.54mm single row")
-    (fp_text reference J7 (at -0.25 -3.6) (layer F.SilkS)
+    (fp_text reference J7 (at -0.127 35.814) (layer F.SilkS)
       (effects (font (size 1 1) (thickness 0.15)))
     )
@@
     (descr "Through hole straight pin header, 1x20, 2.54mm pitch, single row")
     (tags "Through hole pin header THT 1x20 2.54mm single row")
-    (fp_text reference J3 (at 0 -2.33) (layer F.SilkS)
+    (fp_text reference J3 (at 0 50.546) (layer F.SilkS)
       (effects (font (size 1 1) (thickness 0.15)))
     )
@@
     )
   )
+  (module MountingHole:MountingHole_3.2mm_M3 (layer F.Cu)
+    (at 257.429 57.023)
+    (descr "Mounting Hole 3.2mm, no annular, M3")
+    (tags "mounting hole 3.2mm no annular m3")
+    (attr virtual)
+    (fp_text reference REF** (at 0 -4.2) (layer F.SilkS) hide
+      (effects (font (size 1 1) (thickness 0.15)))
+    )
+    (fp_text value MountingHole_3.2mm_M3 (at 0 4.2) (layer F.Fab)
+      (effects (font (size 1 1) (thickness 0.15)))
+    )
+    (fp_circle (center 0 0) (end 3.45 0) (layer F.CrtYd) (width 0.05))
+    (fp_circle (center 0 0) (end 3.2 0) (layer Cmts.User) (width 0.15))
+    (fp_text user %R (at 0.3 0) (layer F.Fab)
+      (effects (font (size 1 1) (thickness 0.15)))
+    )
+    (pad 1 np_thru_hole circle (at 0 0) (size 3.2 3.2) (drill 3.2) (layers *.Cu *.Mask))
+  )
+  (module MountingHole:MountingHole_3.2mm_M3 (layer F.Cu)
+    (at 181.864 57.023)
+    (descr "Mounting Hole 3.2mm, no annular, M3")
+    (tags "mounting hole 3.2mm no annular m3")
+    (attr virtual)
+    (fp_text reference REF** (at 0 -4.2) (layer F.SilkS) hide
+      (effects (font (size 1 1) (thickness 0.15)))
+    )
+    (fp_text value MountingHole_3.2mm_M3 (at 0 4.2) (layer F.Fab)
+      (effects (font (size 1 1) (thickness 0.15)))
+    )
+    (fp_circle (center 0 0) (end 3.45 0) (layer F.CrtYd) (width 0.05))
+    (fp_circle (center 0 0) (end 3.2 0) (layer Cmts.User) (width 0.15))
+    (fp_text user %R (at 0.3 0) (layer F.Fab)
+      (effects (font (size 1 1) (thickness 0.15)))
+    )
+    (pad 1 np_thru_hole circle (at 0 0) (size 3.2 3.2) (drill 3.2) (layers *.Cu *.Mask))
+  )
+  (module MountingHole:MountingHole_3.2mm_M3 (layer F.Cu)
+    (at 181.864 145.669)
+    (descr "Mounting Hole 3.2mm, no annular, M3")
+    (tags "mounting hole 3.2mm no annular m3")
+    (attr virtual)
+    (fp_text reference REF** (at 0 -4.2) (layer F.SilkS) hide
+      (effects (font (size 1 1) (thickness 0.15)))
+    )
+    (fp_text value MountingHole_3.2mm_M3 (at 0 4.2) (layer F.Fab)
+      (effects (font (size 1 1) (thickness 0.15)))
+    )
+    (fp_circle (center 0 0) (end 3.45 0) (layer F.CrtYd) (width 0.05))
+    (fp_circle (center 0 0) (end 3.2 0) (layer Cmts.User) (width 0.15))
+    (fp_text user %R (at 0.3 0) (layer F.Fab)
+      (effects (font (size 1 1) (thickness 0.15)))
+    )
+    (pad 1 np_thru_hole circle (at 0 0) (size 3.2 3.2) (drill 3.2) (layers *.Cu *.Mask))
+  )
+  (module MountingHole:MountingHole_3.2mm_M3 (layer F.Cu)
+    (at 257.429 145.669)
+    (descr "Mounting Hole 3.2mm, no annular, M3")
+    (tags "mounting hole 3.2mm no annular m3")
+    (attr virtual)
+    (fp_text reference REF** (at 0 -4.2) (layer F.SilkS) hide
+      (effects (font (size 1 1) (thickness 0.15)))
+    )
+    (fp_text value MountingHole_3.2mm_M3 (at 0 4.2) (layer F.Fab)
+      (effects (font (size 1 1) (thickness 0.15)))
+    )
+    (fp_circle (center 0 0) (end 3.45 0) (layer F.CrtYd) (width 0.05))
+    (fp_circle (center 0 0) (end 3.2 0) (layer Cmts.User) (width 0.15))
+    (fp_text user %R (at 0.3 0) (layer F.Fab)
+      (effects (font (size 1 1) (thickness 0.15)))
+    )
+    (pad 1 np_thru_hole circle (at 0 0) (size 3.2 3.2) (drill 3.2) (layers *.Cu *.Mask))
+  )
+  (gr_arc (start 180.086 147.447) (end 178.308 147.447) (angle -90) (layer Edge.Cuts) (width 0.15))
+  (gr_arc (start 180.086 55.245) (end 180.086 53.467) (angle -90) (layer Edge.Cuts) (width 0.15))
+  (gr_arc (start 259.207 55.245) (end 260.985 55.245) (angle -90) (layer Edge.Cuts) (width 0.15))
+  (gr_arc (start 259.207 147.447) (end 259.207 149.225) (angle -90) (layer Edge.Cuts) (width 0.15))
   (gr_text "Teensy ++ 2.0" (at 201.676 112.649) (layer F.SilkS)
     (effects (font (size 1.5 1.5) (thickness 0.3)))
@@
     (effects (font (size 1.5 1.5) (thickness 0.3)))
   )
-  (gr_text "BY: Jonathan Low" (at 189.738 143.129) (layer F.SilkS)
-    (effects (font (size 1.5 1.5) (thickness 0.3)))
-  )
-  (gr_text "TP-Keyboard Test Board v1.0" (at 196.469 140.208) (layer F.SilkS)
+  (gr_text "BY: Jonathan Low" (at 198.12 147.066) (layer F.SilkS)
+    (effects (font (size 1.5 1.5) (thickness 0.3)))
+  )
+  (gr_text "TP-Keyboard Test Board v1.0" (at 204.851 144.145) (layer F.SilkS)
     (effects (font (size 1.5 1.5) (thickness 0.3)))
   )
@@
     (effects (font (size 1.25 1.25) (thickness 0.2)))
   )
-  (gr_text 28 (at 257.048 56.261) (layer F.SilkS)
-    (effects (font (size 1.5 1.5) (thickness 0.3)))
-  )
-  (gr_text 27 (at 258.953 60.452) (layer F.SilkS)
-    (effects (font (size 1.5 1.5) (thickness 0.3)))
-  )
-  (gr_text "BY: Jonathan Low\n" (at 189.484 143.383) (layer F.Cu)
-    (effects (font (size 1.5 1.5) (thickness 0.3)))
-  )
-  (gr_text "TP-Keyboard Test Board v1.0" (at 196.215 140.462) (layer F.Cu)
-    (effects (font (size 1.5 1.5) (thickness 0.3)))
-  )
-  (gr_line (start 260.985 53.467) (end 260.985 149.225) (layer Edge.Cuts) (width 0.15))
-  (gr_line (start 178.308 149.225) (end 260.985 149.225) (layer Edge.Cuts) (width 0.15))
-  (gr_line (start 178.308 53.467) (end 178.308 149.225) (layer Edge.Cuts) (width 0.15))
-  (gr_line (start 260.985 53.467) (end 178.308 53.467) (layer Edge.Cuts) (width 0.15))
+  (gr_text "BY: Jonathan Low\n" (at 197.866 147.32) (layer F.Cu)
+    (effects (font (size 1.5 1.5) (thickness 0.3)))
+  )
+  (gr_text "TP-Keyboard Test Board v1.0" (at 204.597 144.399) (layer F.Cu)
+    (effects (font (size 1.5 1.5) (thickness 0.3)))
+  )
+  (gr_line (start 260.985 55.245) (end 260.985 147.447) (layer Edge.Cuts) (width 0.15))
+  (gr_line (start 180.086 149.225) (end 259.207 149.225) (layer Edge.Cuts) (width 0.15))
+  (gr_line (start 178.308 55.245) (end 178.308 147.447) (layer Edge.Cuts) (width 0.15))
+  (gr_line (start 259.207 53.467) (end 180.086 53.467) (layer Edge.Cuts) (width 0.15))
   (segment (start 193.929 59.944) (end 184.912 59.944) (width 0.25) (layer B.Cu) (net 1))
   (segment (start 184.912 62.484) (end 193.929 62.484) (width 0.25) (layer B.Cu) (net 2))

Commit message: replaced with correct 30 pin ffc
Parts:
- removed REF** (x4): MountingHole_3.2mm_M3, MountingHole:MountingHole_3.2mm_M3
- J1: value Conn_01x28_Female -> Conn_01x30_Female; footprint custom:Con_FFC_28_ALT -> custom:Con_FFC_30_2.0mm
- J7: value Conn_01x28_Male -> Conn_01x30_Male; footprint custom:Heade2.54m_28pin -> custom:Heade2.54m_30pin_working
- moved J1 8.58 mm to (255.6, 93.3)
- moved J7 8.58 mm to (240.2, 67.8)
Routing:
- net Net-(J1-Pad29): track 0.00 -> 27.5 mm
- net Net-(J1-Pad13): track 62.6 -> 85.0 mm
- net Net-(J1-Pad27): track 15.9 -> 35.9 mm
- net Net-(J1-Pad30): track 0.00 -> 13.7 mm
- net Net-(J1-Pad7): track 38.1 -> 51.3 mm
- net Net-(J1-Pad5): track 31.7 -> 44.6 mm
- net Net-(J1-Pad3): track 25.3 -> 38.0 mm
- net Net-(J1-Pad15): track 66.4 -> 77.1 mm
- net Net-(J1-Pad19): track 53.4 -> 63.6 mm
- net Net-(J1-Pad11): track 56.2 -> 65.8 mm
- net Net-(J1-Pad17): track 60.0 -> 69.6 mm
- net Net-(J1-Pad23): track 40.3 -> 49.6 mm
- net Net-(J1-Pad21): track 46.8 -> 55.5 mm
- net Net-(J1-Pad9): track 49.8 -> 58.1 mm
- net Net-(J1-Pad25): track 35.0 -> 42.1 mm
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Other:
- board text added: "29"
- board text added: "30"
- board text added: "30 Pin FFC Connector"
- board text removed: "28 Pin FFC Connector"

Commit message: removed footprints further from edge of board
Parts:
- moved J1 0.67 mm to (254.9, 93.3)
- moved J7 0.67 mm to (239.5, 67.8)
