File: pcb/board/board.kicad_pcb (KiCad board)
At the start: 2 copper layers, 31.4 x 53.3 mm, 9 parts, among them J2 RGB LEDs, J3 30 Pin FFC, U1 Teensy++2.0

Commit message: need to move ffc to other side
Parts:
- moved J3 35.8 mm to (175.8, 79.4)
Routing:
- net FFC29: track 0.01 -> 30.1 mm, vias 0 -> 1

Commit message: double check positioning, is a 2nd board necessary?
Parts:
- moved J3 7.32 mm to (177.6, 86.5)
Changed lines of the file:
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@@
   )
   (module custom:Con_FFC_30_2.0mm (layer F.Cu)
-    (at 175.8 79.4 180)
+    (at 177.6 86.5 180)
     (descr "Through hole straight pin header, 1x14, 2.00mm pitch, single row")
     (tags "Through hole pin header THT 1x14 2.00mm single row")
