File: pcb - Copy/board/board.kicad_pcb (KiCad board)
At the start: 2 copper layers, 90.5 x 87 mm, 12 parts, among them J1 Trackpoint, J2 RGB LEDs, J3 30 Pin FFC, U1 Teensy++2.0

Commit message: added led for caps lock indicator
Parts:
- added D1: LED, LED_SMD:LED_1206_3216Metric_Pad1.42x1.75mm_HandSolder, F.Cu at (130.8, 122.6)
- added R3: R, Resistor_SMD:R_1206_3216Metric_Pad1.42x1.75mm_HandSolder, F.Cu at (135.3, 121.1)
- moved R2 42.3 mm to (170.8, 138.6), turned to 180 degrees
- moved J1 28.8 mm to (164.1, 135.2)
- moved R1 16.0 mm to (146.9, 130.9), turned to 90 degrees
Connections:
- U1 pad 47: Net-(U1-Pad47) -> CAPS
Routing:
- net DATA: track 64.3 -> 105.5 mm
- net CLK: track 57.2 -> 85.9 mm
- net 5V: track 93.4 -> 119.5 mm
- net CAPS: track 0.00 -> 15.5 mm, vias 0 -> 2
- net Net-(D1-Pad2): track 0.00 -> 3.02 mm
- net GND: vias 0 -> 6
