File: pcb - Copy/board/board.kicad_pcb (KiCad board)
At the start: 2 copper layers, 90.5 x 87 mm, 14 parts, among them J1 Trackpoint, J2 RGB LEDs, J3 30 Pin FFC, U1 Teensy++2.0

Commit message: figured out pinout of L420 trackpoint, added 8 pin FFC conn. to PCB
Parts:
- added J4: Conn_01x08_Male, custom:FFC_8_TE, F.Cu at (188.5, 143.1)
- moved REF** 14.7 mm to (201.6, 147.0)
- moved REF** 10.4 mm to (118.1, 147.0)
Routing:
- net CLK: track 85.9 -> 120.0 mm
- net DATA: track 105.5 -> 133.2 mm
- net 5V: track 119.5 -> 134.6 mm
- net GND: track 0.00 -> 4.71 mm, vias 6 -> 11
Other:
- board size 90.5 x 87 mm -> 90.5 x 97.3 mm

Commit message: added reset circuit to pcb
Parts:
- added C1: 2.2uF, Capacitor_SMD:C_1206_3216Metric_Pad1.42x1.75mm_HandSolder, F.Cu at (186.7, 134.5)
- added R4: 100K, Resistor_SMD:R_1206_3216Metric_Pad1.42x1.75mm_HandSolder, F.Cu at (180.3, 134.5)
Routing:
- net RST: track 0.00 -> 19.1 mm
- net 5V: track 134.6 -> 141.1 mm
- net GND: vias 11 -> 14
Changed lines of the file:
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@@
     (thickness 1.6)
     (drawings 20)
-    (tracks 286)
+    (tracks 300)
     (zones 0)
-    (modules 15)
+    (modules 17)
     (nets 55)
   )
@@
     (pad 0 smd rect (at 5.334 5.2324) (size 1.2 1.8) (layers F.Cu F.Paste F.Mask))
   )
+  (module Capacitor_SMD:C_1206_3216Metric_Pad1.42x1.75mm_HandSolder (layer F.Cu)
+    (at 186.7 134.5)
+    (descr "Capacitor SMD 1206 (3216 Metric), square (rectangular) end terminal, IPC_7351 nominal with elongated pad for handsoldering. (Body size source: http://www.tortai-tech.com/upload/download/2011102023233369053.pdf), generated with kicad-footprint-generator")
+    (tags "capacitor handsolder")
+    (attr smd)
+    (fp_text reference C1 (at 0 -1.82) (layer F.SilkS)
+      (effects (font (size 1 1) (thickness 0.15)))
+    )
+    (fp_text value 2.2uF (at 0 1.82) (layer F.Fab)
+      (effects (font (size 1 1) (thickness 0.15)))
+    )
+    (fp_line (start -1.6 0.8) (end -1.6 -0.8) (layer F.Fab) (width 0.1))
+    (fp_line (start -1.6 -0.8) (end 1.6 -0.8) (layer F.Fab) (width 0.1))
+    (fp_line (start 1.6 -0.8) (end 1.6 0.8) (layer F.Fab) (width 0.1))
+    (fp_line (start 1.6 0.8) (end -1.6 0.8) (layer F.Fab) (width 0.1))
+    (fp_line (start -0.602064 -0.91) (end 0.602064 -0.91) (layer F.SilkS) (width 0.12))
+    (fp_line (start -0.602064 0.91) (end 0.602064 0.91) (layer F.SilkS) (width 0.12))
+    (fp_line (start -2.45 1.12) (end -2.45 -1.12) (layer F.CrtYd) (width 0.05))
+    (fp_line (start -2.45 -1.12) (end 2.45 -1.12) (layer F.CrtYd) (width 0.05))
+    (fp_line (start 2.45 -1.12) (end 2.45 1.12) (layer F.CrtYd) (width 0.05))
+    (fp_line (start 2.45 1.12) (end -2.45 1.12) (layer F.CrtYd) (width 0.05))
+    (fp_text user %R (at 0 0) (layer F.Fab)
+      (effects (font (size 0.8 0.8) (thickness 0.12)))
+    )
+    (pad 1 smd roundrect (at -1.4875 0) (size 1.425 1.75) (layers F.Cu F.Paste F.Mask) (roundrect_rratio 0.175439)
+      (net 1 5V))
+    (pad 2 smd roundrect (at 1.4875 0) (size 1.425 1.75) (layers F.Cu F.Paste F.Mask) (roundrect_rratio 0.175439)
+      (net 54 RST))
+    (model ${KISYS3DMOD}/Capacitor_SMD.3dshapes/C_1206_3216Metric.wrl
+      (at (xyz 0 0 0))
+      (scale (xyz 1 1 1))
+      (rotate (xyz 0 0 0))
+    )
+  )
+  (module Resistor_SMD:R_1206_3216Metric_Pad1.42x1.75mm_HandSolder (layer F.Cu)
+    (at 180.2875 134.5)
+    (descr "Resistor SMD 1206 (3216 Metric), square (rectangular) end terminal, IPC_7351 nominal with elongated pad for handsoldering. (Body size source: http://www.tortai-tech.com/upload/download/2011102023233369053.pdf), generated with kicad-footprint-generator")
+    (tags "resistor handsolder")
+    (attr smd)
+    (fp_text reference R4 (at 0 -1.82) (layer F.SilkS)
+      (effects (font (size 1 1) (thickness 0.15)))
+    )
+    (fp_text value 100K (at 0 1.82) (layer F.Fab)
+      (effects (font (size 1 1) (thickness 0.15)))
+    )
+    (fp_line (start -1.6 0.8) (end -1.6 -0.8) (layer F.Fab) (width 0.1))
+    (fp_line (start -1.6 -0.8) (end 1.6 -0.8) (layer F.Fab) (width 0.1))
+    (fp_line (start 1.6 -0.8) (end 1.6 0.8) (layer F.Fab) (width 0.1))
+    (fp_line (start 1.6 0.8) (end -1.6 0.8) (layer F.Fab) (width 0.1))
+    (fp_line (start -0.602064 -0.91) (end 0.602064 -0.91) (layer F.SilkS) (width 0.12))
+    (fp_line (start -0.602064 0.91) (end 0.602064 0.91) (layer F.SilkS) (width 0.12))
+    (fp_line (start -2.45 1.12) (end -2.45 -1.12) (layer F.CrtYd) (width 0.05))
+    (fp_line (start -2.45 -1.12) (end 2.45 -1.12) (layer F.CrtYd) (width 0.05))
+    (fp_line (start 2.45 -1.12) (end 2.45 1.12) (layer F.CrtYd) (width 0.05))
+    (fp_line (start 2.45 1.12) (end -2.45 1.12) (layer F.CrtYd) (width 0.05))
+    (fp_text user %R (at 0 0) (layer F.Fab)
+      (effects (font (size 0.8 0.8) (thickness 0.12)))
+    )
+    (pad 1 smd roundrect (at -1.4875 0) (size 1.425 1.75) (layers F.Cu F.Paste F.Mask) (roundrect_rratio 0.175439)
+      (net 2 GND))
+    (pad 2 smd roundrect (at 1.4875 0) (size 1.425 1.75) (layers F.Cu F.Paste F.Mask) (roundrect_rratio 0.175439)
+      (net 54 RST))
+    (model ${KISYS3DMOD}/Resistor_SMD.3dshapes/R_1206_3216Metric.wrl
+      (at (xyz 0 0 0))
+      (scale (xyz 1 1 1))
+      (rotate (xyz 0 0 0))
+    )
+  )
   (dimension 97.4 (width 0.12) (layer F.SilkS)
     (gr_text "97.400 mm" (at 73.43 101.8 270) (layer F.SilkS)
@@
   (segment (start 172.2875 137.725) (end 169.7625 135.2) (width 0.4) (layer F.Cu) (net 1))
   (segment (start 172.2875 138.6) (end 172.2875 137.725) (width 0.4) (layer F.Cu) (net 1))
+  (segment (start 181.5 138.6) (end 182.9 138.6) (width 0.4) (layer F.Cu) (net 1))
+  (segment (start 185.2125 136.2875) (end 185.2125 134.5) (width 0.4) (layer F.Cu) (net 1))
+  (segment (start 182.9 138.6) (end 185.2125 136.2875) (width 0.4) (layer F.Cu) (net 1))
   (via (at 125 119.3) (size 2) (drill 1) (layers F.Cu B.Cu) (net 2))
   (via (at 128.3 119.3) (size 2) (drill 1) (layers F.Cu B.Cu) (net 2))
@@
   (via (at 189.4 140.1) (size 0.8) (drill 0.4) (layers F.Cu B.Cu) (net 2))
   (via (at 187.4 138.3) (size 0.8) (drill 0.4) (layers F.Cu B.Cu) (net 2))
+  (via (at 177.2 134.5) (size 0.8) (drill 0.4) (layers F.Cu B.Cu) (net 2))
+  (via (at 177.2 133.5) (size 0.8) (drill 0.4) (layers F.Cu B.Cu) (net 2))
+  (via (at 177.2 135.5) (size 0.8) (drill 0.4) (layers F.Cu B.Cu) (net 2))
   (segment (start 157.62 133.8) (end 159.02 135.2) (width 0.2) (layer F.Cu) (net 3))
   (segment (start 117.2 115.6) (end 135.4 133.8) (width 0.2) (layer F.Cu) (net 3))
@@
   (segment (start 132.3 108.67) (end 130.34 106.71) (width 0.2) (layer F.Cu) (net 50))
   (segment (start 132.3 109.6) (end 132.3 108.67) (width 0.2) (layer F.Cu) (net 50))
+  (segment (start 188.9 134.5) (end 188.1875 134.5) (width 0.2) (layer F.Cu) (net 54))
+  (segment (start 191 136.6) (end 188.9 134.5) (width 0.2) (layer F.Cu) (net 54))
+  (segment (start 191 143.1) (end 191 136.6) (width 0.2) (layer F.Cu) (net 54))
+  (segment (start 188.1875 133.625) (end 187.2625 132.7) (width 0.2) (layer F.Cu) (net 54))
+  (segment (start 188.1875 134.5) (end 188.1875 133.625) (width 0.2) (layer F.Cu) (net 54))
+  (segment (start 181.775 133.625) (end 181.775 134.5) (width 0.2) (layer F.Cu) (net 54))
+  (segment (start 182.7 132.7) (end 181.775 133.625) (width 0.2) (layer F.Cu) (net 54))
+  (segment (start 187.2625 132.7) (end 182.7 132.7) (width 0.2) (layer F.Cu) (net 54))
   (zone (net 2) (net_name GND) (layer F.Cu) (hatch edge 0.508)
     (connect_pads (clearance 0.508))
